Commit message: fix odom drifting: correct laser

File: robot_nav/urdf/robot_descript.urdf (robot description, URDF)
Before this commit: robot bot, 7 links, 6 joints
Joints:
- joint dummy_joint: origin (none) -> xyz=0 0 0.076 rpy=0 0 0

File: robot_slam/urdf/robot_descript.urdf (robot description, URDF)
Before this commit: robot bot, 7 links, 6 joints
Joints:
- joint dummy_joint: origin (none) -> xyz=0 0 0.076 rpy=0 0 0
